Commit message: remove that jitter

File: kr5_description/urdf/braccio_planning_model.urdf (robot description, URDF)
Before this commit: robot kr5, 9 links, 8 joints
Links:
- link base_link: geometry visual cylinder length=0.01 radius=.053

Commit message: both grippers independent

File: kr5_description/urdf/braccio_planning_model.urdf (robot description, URDF)
Before this commit: robot kr5, 9 links, 8 joints
Joints:
- joint sub_gripper_joint: limit lower=1.2741 upper=2.3732 effort=1.0 velocity=1.0 -> lower=0.1750 upper=1.2741 effort=1.0 velocity=1.0; mimic joint=gripper_joint -> (none)
