Commit message: pickin up the box woohoo

File: braccio_description/urdf/braccio_planning_model.urdf (robot description, URDF)
Before this commit: robot kr5, 9 links, 8 joints
Joints:
- joint gripper_joint: limit lower=0.1750 upper=1.2741 effort=1.0 velocity=1.0 -> lower=0.1750 upper=1.2741 effort=1000.0 velocity=1.0
- joint joint_a1: limit lower=0.0 upper=3.1416 effort=1.0 velocity=1.0 -> lower=0.0 upper=3.1416 effort=1000.0 velocity=1.0
- joint joint_a2: limit lower=0.2618 upper=2.8798 effort=1.0 velocity=1.0 -> lower=0.2618 upper=2.8798 effort=1000.0 velocity=1.0
- joint joint_a3: limit lower=0 upper=3.1416 effort=1.0 velocity=1.0 -> lower=0 upper=3.1416 effort=1000.0 velocity=1.0
- joint joint_a4: limit lower=0 upper=3.1416 effort=1.0 velocity=1.0 -> lower=0 upper=3.1416 effort=1000.0 velocity=1.0
- joint joint_a5: limit lower=0.0 upper=3.1416 effort=1.0 velocity=1.0 -> lower=0.0 upper=3.1416 effort=1000.0 velocity=1.0
- joint sub_gripper_joint: limit lower=0.1750 upper=1.2741 effort=1.0 velocity=1.0 -> lower=0.1750 upper=1.2741 effort=1000.0 velocity=1.0

Commit message: rample tumble into bowl

File: braccio_description/urdf/braccio_planning_model.urdf (robot description, URDF)
Before this commit: robot kr5, 9 links, 8 joints
Joints:
- joint gripper_joint: limit lower=0.1750 upper=1.2741 effort=1000.0 velocity=1.0 -> lower=0.1750 upper=1.2741 effort=10.0 velocity=1.0
- joint sub_gripper_joint: limit lower=0.1750 upper=1.2741 effort=1000.0 velocity=1.0 -> lower=0.1750 upper=1.2741 effort=10.0 velocity=1.0

Commit message: sort of almost works irl

File: braccio_description/urdf/braccio_planning_model.urdf (robot description, URDF)
Before this commit: robot kr5, 9 links, 8 joints
Joints:
- removed joint joint_a1
- removed joint joint_a2
- removed joint joint_a3
- removed joint joint_a4
- removed joint joint_a5
- added joint base_joint: type revolute, parent base_link, child link_1, origin xyz=0 0 0 rpy=0 0 0, axis 0 0 -1, limit lower=0.0 upper=3.1416 effort=1000.0 velocity=1.0
- added joint elbow_joint: type revolute, parent link_2, child link_3, origin xyz=0 0 0.125 rpy=-1.5708 0 0, axis 1 0 0, limit lower=0 upper=3.1416 effort=1000.0 velocity=1.0
- added joint shoulder_joint: type revolute, parent link_1, child link_2, origin xyz=0 -.002 0.072 rpy=-1.5708 0 0, axis 1 0 0, limit lower=0.2618 upper=2.8798 effort=1000.0 velocity=1.0
- added joint wrist_pitch_joint: type revolute, parent link_3, child link_4, origin xyz=0 0 0.125 rpy=-1.5708 0 0, axis 1 0 0, limit lower=0 upper=3.1416 effort=1000.0 velocity=1.0
- added joint wrist_roll_joint: type revolute, parent link_4, child link_5, origin xyz=0 0.0 0.06 rpy=0 0 1.5708, axis 0 0 -1, limit lower=0.0 upper=3.1416 effort=1000.0 velocity=1.0

Commit message: updated for cooking robot

File: braccio_description/urdf/braccio_planning_model.urdf (robot description, URDF)
Before this commit: robot kr5, 9 links, 8 joints
Links:
- link right_gripper_link: geometry collision mesh filename=package://braccio_description/stl/braccio_left_gripper.stl scale=0.001 0.001 0.001; visual mesh filename=package://braccio_description/stl/braccio_right_gripper.stl scale=0.001 0.001 0.001
